Commit message: detect zone ball order

File: gillou/src/description/gillou.urdf (robot description, URDF)
Before this commit: robot gillou_bot, 13 links, 12 joints
Links:
- link first_hook_link: geometry collision cylinder length=${hook_width} radius=${hook_radius}; visual cylinder length=${hook_width} radius=${hook_radius}
